Commit message: navigation + slam + amcl first test

File: ws/src/willy/description/urdf/willy.urdf.xacro (robot description, xacro)
@@ -3,3 +3,4 @@
   <xacro:include filename="willy_core.xacro" />
   <xacro:include filename="gazebo_control.xacro" />
+  <xacro:include filename="lidar.xacro" />
 </robot>

File: ws/src/willy/description/urdf/willy_core.xacro (robot description, xacro)
@@ -14,6 +14,17 @@
         <color rgba="0 0 0 1" />
     </material>
+    <material name="red">
+        <color rgba="1 0 0 1" />
+    </material>
     <!-- BASE LINK -->
     <link name="base_link">
+    </link>
+    <!-- BASE_FOOTPRINT LINK -->
+    <joint name="base_footprint_joint" type="fixed">
+        <parent link="base_footprint"/>
+        <child link="base_link"/>
+        <origin xyz="0 0 0" rpy="0 0 0"/>
+    </joint>
+    <link name="base_footprint">
     </link>
     <!-- CHASSIS LINK -->
